File: FC PCB/ELRSFC.kicad_pcb (KiCad board)
At the start: 2 copper layers, 33 x 33 mm, 82 parts, among them SW1 SWITCH, SW2 SWITCH, U1 W25Q128JVSIQTR, U2 XL1509-5.0E1, U3 AMS1117-3.3, U4 AT7456E, U5 MPU6500, U6 STM32F411CEU6, X2 27MHz, X3 25MHz

Commit message: Seventh entry
Parts:
- added C17: 0.1uF, Capacitor_SMD:C_0402_1005Metric, F.Cu at (135.9, 46.6)
- added C23: 0.1uF, Capacitor_SMD:C_0402_1005Metric, F.Cu at (135.9, 48.6)
- added C24: 10nF, Capacitor_SMD:C_0402_1005Metric, F.Cu at (135.9, 50.5)
- added C25: 470nF, Capacitor_SMD:C_0603_1608Metric, F.Cu at (131.1, 52.9)
- added C26: 10nF, Capacitor_SMD:C_0402_1005Metric, F.Cu at (135.9, 52.5)
- added C31: 10pF, Capacitor_SMD:C_0402_1005Metric, F.Cu at (150.2, 80.6)
- added C33: 10pF, Capacitor_SMD:C_0402_1005Metric, F.Cu at (152.2, 78.8)
- added C47: 0.1uF, Capacitor_SMD:C_0402_1005Metric, F.Cu at (148.8, 80.3)
- added C48: 0.1uF, Capacitor_SMD:C_0402_1005Metric, F.Cu at (148.9, 81.8)
- added C49: 10uF, Capacitor_SMD:C_0402_1005Metric, F.Cu at (156.1, 92.8)
- added C50: 0.1uF, Capacitor_SMD:C_0402_1005Metric, F.Cu at (150.6, 58.7)
- added FL1: 2450FM07D0034T, ELRSFC:FIL_2450FM07D0034T, F.Cu at (125.4, 52.8)
- added J1: Conn_Coaxial_Small, Connector_Coaxial:U.FL_Hirose_U.FL-R-SMT-1_Vertical, F.Cu at (128.0, 58.0)
- added JP1: ENA, ELRSFC:ENA, F.Cu at (156.7, 49.1)
- added JP2: FLASH, ELRSFC:FLASH, F.Cu at (156.7, 51.7)
- added R14: 12k, Resistor_SMD:R_0402_1005Metric, F.Cu at (153.5, 48.8)
- added R15: 10k, Resistor_SMD:R_0402_1005Metric, F.Cu at (153.5, 50.8)
- added R16: 10k, Resistor_SMD:R_0402_1005Metric, F.Cu at (153.5, 52.8)
- added U7: ESP8285H16, ELRSFC:QFN-32_L5.0-W5.0-P0.50-TL-EP3.7, F.Cu at (151.5, 84.9)
- added U8: SX1281IMLTRT, ELRSFC:QFN-24_L4.0-W4.0-P0.50-TL-EP2.6, F.Cu at (159.8, 88.5)
- added X1: 52MHz, ELRSFC:CRYSTAL-SMD_4P-L2.0-W1.6-BL, F.Cu at (163.5, 86.8)
- added X4: 26MHz, ELRSFC:CRYSTAL-SMD_4P-L2.0-W1.6-BL, F.Cu at (152.2, 80.6)
- SW1, SW2: footprint ELRSFC:SW-SMD_L3.9-W3.0-P4.45 -> ELRSFC:SW_TS-1187A-B-A-B
- moved R10 41.3 mm to (162.9, 82.3), turned to 90 degrees
- moved C35 32.8 mm to (159.8, 66.1)
- moved C21 32.1 mm to (159.9, 63.4)
- moved R6 24.5 mm to (143.0, 74.2)
- moved D4 23.0 mm to (144.8, 82.0), turned to 180 degrees
- moved D3 20.1 mm to (143.4, 76.1), turned to 180 degrees
- moved SW2 15.0 mm to (157.6, 95.1)
- moved SW1 14.8 mm to (165.7, 95.4)
- moved U2 0.36 mm to (169.1, 64.3)
- moved U1 0.16 mm to (170.6, 72.0)
- moved X3 0.14 mm to (156.9, 82.7)
Connections:
- C27 pad 1: GND -> +5V
- C27 pad 2: +5V -> GND
- C28 pad 1: GND -> +5V
- C28 pad 2: +5V -> GND
- C29 pad 1: GND -> +5V
- C29 pad 2: +5V -> GND
- U4 pad 29: unconnected-(U4-EP-Pad29) -> GND
- U6 pad 49: +3v3 -> GND
Routing:
- net GND: track 14.6 -> 43.9 mm, vias 1 -> 3
- net GPIO5: track 0.00 -> 9.43 mm
- net GPIO4: track 0.00 -> 8.90 mm
- net Net-(U7-XTAL_OUT): track 0.00 -> 4.17 mm
- net +3v3: track 8.30 -> 12.3 mm, vias 2 -> 4
- net Net-(U6-PH0-OSC_IN): track 0.00 -> 3.81 mm
- net Net-(U8-XTA): track 0.00 -> 2.96 mm
- net Net-(U7-XTAL_IN): track 0.00 -> 2.65 mm
- net Net-(U8-XTB): track 0.00 -> 2.01 mm
- net Net-(U6-PH1-OSC_OUT): track 0.00 -> 1.92 mm

Commit message: Eight entry
Parts:
- H5, H7, H9, JP1, JP2: moved to B.Cu
- J1: footprint Connector_Coaxial:U.FL_Hirose_U.FL-R-SMT-1_Vertical -> ELRSFC:UFL
- moved FL1 53.2 mm to (163.0, 90.4)
- moved C17 50.8 mm to (156.3, 93.0), turned to 180 degrees
- moved J1 50.1 mm to (166.2, 90.4), turned to -90 degrees
- moved C23 47.7 mm to (154.5, 92.5), turned to 180 degrees
- moved C24 45.1 mm to (156.2, 90.8), turned to 180 degrees
- moved C25 44.6 mm to (160.2, 86.7), turned to 90 degrees
- moved C26 43.6 mm to (161.5, 87.8), turned to 90 degrees
- moved R16 37.0 mm to (155.2, 89.8)
- moved R10 36.0 mm to (136.1, 58.3), turned to 0 degrees
- moved C50 29.4 mm to (148.5, 88.0), turned to -90 degrees
- moved SW1 26.5 mm to (139.2, 94.3)
- moved SW2 23.1 mm to (134.5, 94.2)
- moved U3 21.9 mm to (191.4, 80.8)
- moved C49 16.5 mm to (148.4, 78.2), turned to 90 degrees
- moved X1 5.89 mm to (157.6, 86.9), turned to 180 degrees
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Routing:
- net GND: track 43.9 -> 74.7 mm, vias 3 -> 109
- net +3v3: track 12.3 -> 33.7 mm, vias 4 -> 6
- net GPIO15: track 0.00 -> 19.2 mm, vias 0 -> 2
- net GPIO14: track 0.00 -> 19.0 mm
- net GPIO13: track 0.00 -> 18.1 mm
- net GPIO12: track 0.00 -> 17.3 mm, vias 0 -> 2
- net Net-(JP2-B): track 0.00 -> 15.4 mm, vias 0 -> 2
- net GPIO2: track 0.00 -> 13.2 mm, vias 0 -> 2
- net DCC_FB: track 0.00 -> 12.0 mm, vias 0 -> 3
- net PA3: track 0.00 -> 10.5 mm, vias 0 -> 2
- net PA2: track 0.00 -> 8.78 mm, vias 0 -> 2
- net GPIO4: track 8.90 -> 5.58 mm
- net Net-(JP1-B): track 0.00 -> 1.97 mm
- net GPIO5: track 9.43 -> 8.03 mm
- net Net-(J1-In): track 0.00 -> 1.10 mm
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- added copper zone on B.Cu, net GND
Other:
- outline, holes or cut-outs redrawn

Commit message: Ninth entry
Parts:
- removed C18: 10uF, Capacitor_SMD:C_0402_1005Metric
- removed C19: 0.1uF, Capacitor_SMD:C_0402_1005Metric
- H4: moved to B.Cu
- H6: value VTX -> GPS
- X2: footprint ELRSFC:CRYSTAL-SMD_4P-L3.2-W2.5-BL -> ELRSFC:CRYSTAL-SMD_4P-L2.0-W1.6-BL
- moved C1 75.1 mm to (180.0, 75.9), turned to -90 degrees
- moved C2 73.4 mm to (178.9, 75.9), turned to -90 degrees
- moved R8 62.5 mm to (177.0, 70.5), turned to 180 degrees
- moved C29 62.2 mm to (177.1, 62.5)
- moved C28 61.2 mm to (175.3, 68.5)
- moved C34 58.6 mm to (175.2, 62.5)
- moved R3 57.4 mm to (177.0, 78.3)
- moved R9 54.7 mm to (165.1, 62.5), turned to 180 degrees
- moved C27 50.9 mm to (165.3, 63.8), turned to 180 degrees
- moved C10 48.9 mm to (159.9, 64.8), turned to 90 degrees
- moved C12 47.2 mm to (158.9, 64.8), turned to 90 degrees
- moved C11 46.5 mm to (157.9, 64.8), turned to 90 degrees
- moved R2 42.1 mm to (161.2, 66.8), turned to 180 degrees
- moved H6 41.6 mm to (179.7, 71.8)
- moved R1 37.9 mm to (157.2, 66.8)
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Routing:
- net +5V: track 6.99 -> 43.3 mm, vias 0 -> 4
- net GND: track 74.7 -> 109.2 mm, vias 109 -> 113
- net PB14: track 0.00 -> 24.6 mm, vias 0 -> 2
- net PB1: track 0.00 -> 19.8 mm, vias 0 -> 2
- net PB15: track 0.00 -> 19.1 mm, vias 0 -> 2
- net PB13: track 0.00 -> 17.1 mm, vias 0 -> 2
- net +3v3: track 33.7 -> 47.9 mm, vias 6 -> 10
- net Net-(U4-VOUT): track 0.00 -> 11.7 mm, vias 0 -> 1
- net BYPASS: track 0.00 -> 10.4 mm, vias 0 -> 1
- net PB12: track 0.00 -> 9.93 mm, vias 0 -> 2
- net VIDIN: track 0.00 -> 9.77 mm, vias 0 -> 1
- net Net-(U4-SAG): track 0.00 -> 8.58 mm, vias 0 -> 1
- net DIN-: track 6.18 -> 12.4 mm
- net VIN: track 0.00 -> 5.97 mm
- net DIN+: track 5.54 -> 11.4 mm
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
Commit message: high cortisol
Parts:
- removed C14, C15, C16, C22, C3: 10uF, Capacitor_SMD:C_0603_1608Metric
- removed C20, C46, C6, C9: 0.1uF, Capacitor_SMD:C_0402_1005Metric
- removed H9: RX, ELRSFC:RX
- removed SW1, SW2: SWITCH, ELRSFC:SW_TS-1187A-B-A-B
- removed U3: AMS1117-3.3, ELRSFC:SOT-223-3_L6.5-W3.4-P2.30-LS7.0-BR
- added C18: 10nF, Capacitor_SMD:C_0402_1005Metric, F.Cu at (162.2, 83.6)
- added REF**: GPS, ELRSFC:DEBUG_RX, B.Cu at (159.9, 81.7)
- added REF**: GPS, ELRSFC:DEBUG_TX, B.Cu at (161.5, 81.8)
- added U9: SPX3819M5-L-3-3/TR, ELRSFC:SOT-23-5_L3.0-W1.7-P0.95-LS2.8-BL, B.Cu at (164.8, 83.1)
- C5: footprint Capacitor_SMD:C_0402_1005Metric -> Capacitor_SMD:C_0603_1608Metric; moved to B.Cu
- H6: value GPS -> VTX
- R4, R7: footprint Resistor_SMD:R_0402_1005Metric -> Resistor_SMD:R_0603_1608Metric; moved to B.Cu
- moved C4 64.4 mm to (167.5, 82.2), turned to 180 degrees
- moved C7 62.6 mm to (168.9, 79.6)
- moved D1 59.9 mm to (173.2, 78.9), turned to 180 degrees
- moved C13 59.1 mm to (167.5, 81.2), turned to 180 degrees
- moved C8 59.0 mm to (162.1, 82.2), turned to 180 degrees
- moved R11 57.4 mm to (179.8, 79.8), turned to 90 degrees
- moved R12 56.3 mm to (178.8, 79.8), turned to -90 degrees
- moved R13 53.1 mm to (174.9, 70.8), turned to 90 degrees
- moved C5 51.1 mm to (154.9, 79.7), turned to 90 degrees
- moved R5 50.6 mm to (169.9, 85.7), turned to 180 degrees
- moved C41 49.8 mm to (160.0, 81.5)
- moved C42 49.2 mm to (160.0, 82.5)
- moved C40 48.7 mm to (160.7, 83.9), turned to -90 degrees
- moved C43 47.4 mm to (157.2, 85.0)
- moved C45 36.5 mm to (154.8, 71.7), turned to 90 degrees
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Connections:
- H7 pad 1: NRST -> BOOT0
- H7 pad 2: PA13 -> NRST
- H7 pad 3: PA14 -> PA13
- U6 pad 2: Net-(D4-K) -> unconnected-(U6-PC13-Pad2)
- U6 pad 29: unconnected-(U6-PA8-Pad29) -> Net-(D4-K)
Routing:
- net +5V: track 43.3 -> 108.2 mm, vias 4 -> 9
- net GND: track 109.2 -> 161.4 mm, vias 113 -> 125
- net +3v3: track 47.9 -> 85.3 mm, vias 10 -> 21
- net PB0: track 0.00 -> 22.2 mm
- net BATTERY: track 0.00 -> 21.8 mm, vias 0 -> 2
- net Net-(JP1-B): track 1.97 -> 22.5 mm, vias 0 -> 2
- net PB2: track 0.00 -> 17.5 mm, vias 0 -> 2
- net PA9: track 0.00 -> 13.6 mm
- net PA10: track 0.00 -> 13.3 mm
- net NRST: track 0.00 -> 10.7 mm, vias 0 -> 1
- net PA13: track 0.00 -> 8.83 mm, vias 0 -> 1
- net Net-(BUZZER1-Pad1): track 0.00 -> 8.59 mm, vias 0 -> 1
- net PB4: track 0.00 -> 7.03 mm
- net PB8: track 0.00 -> 6.32 mm
- net Net-(JP2-B): track 15.4 -> 21.4 mm, vias 2 -> 1
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
Commit message: (hopefully) finalized PCB
Parts:
- added D5: 1N4148W, Diode_SMD:D_SOD-123, B.Cu at (179.4, 71.2)
- added H10: SENSE, ELRSFC:SENSE, B.Cu at (164.6, 77.3)
- added H9: EXTRA, ELRSFC:EXTRA, B.Cu at (152.8, 70.2)
- added Q1: 2N7002, Package_TO_SOT_SMD:SOT-23, B.Cu at (178.1, 75.6)
- added R17: 10k, Resistor_SMD:R_0402_1005Metric, F.Cu at (176.4, 71.8)
- H5: moved to F.Cu
- moved C39 0.82 mm to (162.5, 74.0)
- moved C44 0.80 mm to (162.8, 72.5)
- moved H7 0.50 mm to (153.8, 72.0)
Connections:
- BUZZER1 pad 1: Net-(BUZZER1-Pad1) -> +3v3
- BUZZER1 pad 2: GND -> Net-(D5-A)
- R13 pad 2: Net-(BUZZER1-Pad1) -> Net-(Q1-G)
- R3 pad 2: PB1 -> PB10
- REF** pad 1: (no net) -> PA3
- REF** pad 1: (no net) -> PA2
- U1 pad 1: PB1 -> PB10
- U6 pad 21: unconnected-(U6-PB10-Pad21) -> PB10
- U6 pad 38: unconnected-(U6-PA15-Pad38) -> PA15
Routing:
- net PB10: track 0.00 -> 19.9 mm
- net Net-(D5-A): track 0.00 -> 18.7 mm
- net PB1: track 20.4 -> 4.11 mm
- net Net-(Q1-G): track 0.00 -> 12.7 mm, vias 0 -> 1
- net Net-(BUZZER1-Pad1): track 8.59 -> 0.00 mm, vias 1 -> 0
- net GND: track 161.4 -> 168.7 mm, vias 125 -> 122
- net PA15: track 0.00 -> 5.23 mm, vias 0 -> 1
- net Net-(C30-Pad2): track 5.67 -> 8.98 mm
- net PB2: track 17.5 -> 18.9 mm
- net +5V: track 108.2 -> 109.2 mm, vias 9 -> 8
Other:
- board text added: "Merlyn411"
