File: FC PCB/ELRSFC.kicad_sch (KiCad schematic)
At the start: 30 parts, among them SW1 SWITCH, U1 STM32F411RET6, U2 AMS1117-5.0, U3 AMS1117-3.3, X1 25MHz

Commit message: Fourth journal entry
Parts:
- removed U2: AMS1117-5.0, lcsc:SOT-223_L6.5-W3.5-P2.30-LS7.0-BR, symbol ELRSFC:AMS1117-5.0
- added C21, C35: 100uF, lcsc:CASE-B_3528, symbol ELRSFC:TAJB107K006RNJ
- added C22, C23, C24, C25, C26: 22uF, symbol Device:C
- added C27, C28, C29, C34: 0.1uF, symbol Device:C
- added C30, C31, C32, C33: 10uF, lcsc:CAP-SMD_L3.2-W1.6-RD-C7171, symbol ELRSFC:TAJA106K016RNJ
- added D1: SS34, Diode_SMD:D_SMA, symbol Diode:SS34
- added D2: GREEN, symbol Device:LED
- added D3: RED, symbol Device:LED
- added L1: 68uH, symbol Device:L
- added R5, R7: 10k, symbol Device:R
- added R6: 5.1k, symbol Device:R
- added R8, R9: 75, symbol Device:R
- added SW2: SWITCH, lcsc:SW-SMD_L3.9-W3.0-P4.45, symbol ELRSFC:TS-1088-AR02016
- added U2: XL1509-5.0E1, lcsc:SOIC-8_L5.0-W4.0-P1.27-LS6.0-BL, symbol ELRSFC:XL1509-5.0E1
- added U4: AT7456E, lcsc:TSSOP-28_L9.7-W4.4-P0.65-LS6.4-BL-EP-2, symbol ELRSFC:AT7456E
- added X2: 27MHz, lcsc:CRYSTAL-SMD_4P-L3.2-W2.5-BL, symbol ELRSFC:S3227000181040
- C13: value 22uF -> 10uF
- C4, C5: value 10uF -> 0.1uF
- C7: value 0.1uF -> 10uF
- R3: value 4.7 -> 5.1k
Connections:
- net +3v3: now also R3.1, R6.1, R7.1
- net +5V: now also C13.1, C21.1, C27.2, C28.2, C29.2, C35.1, L1.2, U2.3 (FB), U4.19 (~{RESET}), U4.21 (AVDD), U4.24 (PVDD), U4.3 (DVDD); no longer C5.1
- net BATTERY: now also C22.1, C23.1, C24.1, C25.1, C26.1, U2.1 (VIN); no longer R3.2
- net GND: now also C5.1, C21.2, C22.2, C23.2, C24.2, C25.2, C26.2, C27.1, C28.1, C29.1, C35.2, D1.2 (A), D3.1 (K), R5.2, R9.2, SW2.2, U2.5 (GND), U2.6 (GND), U2.7 (GND), U2.8 (GND), U4.20 (AGND), U4.23 (PGND), U4.4 (DGND), X2.2 (GND), X2.4 (GND); no longer C5.2
- net at U1.2 (PC13): now also D2.1 (K)
- net PB12: now reaches U1.33 (PB12)
- net PB12: now also U4.8 (~{CS})
- net PB13: now reaches U1.34 (PB13)
- net PB13: now also U4.10 (SCLK)
- net PB14: now reaches U1.35 (PB14)
- net PB14: now also U4.11 (SDOUT)
- net PB15: now reaches U1.36 (PB15)
- net PB15: now also U4.9 (SDIN)
- net NRST: now reaches U1.7 (NRST)
- net NRST: now also C5.2, R7.2, SW2.1
- new net: R5.1, U2.4 (ON/OFF)
- new net: C30.1, C31.1, U4.25 (SAG)
- new net: C32.1, C33.1, U4.26 (VOUT)
- new net: U4.5 (CLKIN), X2.3 (OSC2)
- new net: U4.6 (XFB), X2.1 (OSC1)
- new net: D1.1 (K), L1.1, U2.2 (OUTPUT)
- new net: C30.2, C31.2, C32.2, C33.2, R8.2
- new net: D3.2 (A), R6.2
- new net: D2.2 (A), R3.2
- new net VIDIN: C34.1, R9.1
- new net VIDOUT: R8.1
- new net VIN: C34.2, U4.22 (VIN)
- no-connect marks 5 -> 17
Other:
- note added: "3.3v Power Regulation"
- note added: "5v Power Regulation"
- note added: "OSD"
- note added: "USB"
- title: (none) -> Merlyn411
- moved on the sheet: C1, C10, C11, C12, C14, C15, C16, C17, C18, C19, C2, C20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

Commit message: Fifth journal entry
Parts:
- removed C23, C24, C25, C26: 22uF, symbol Device:C
- removed D2: GREEN, symbol Device:LED
- removed U1: STM32F411RET6, lcsc:LQFP-64_L10.0-W10.0-P0.50-LS12.0-BL, symbol ELRSFC:STM32F411RET6
- removed X1: 25MHz, lcsc:CRYSTAL-SMD_4P-L3.2-W2.5-BL, symbol ELRSFC:X322525MOB4SI
- added BUZZER1: BUZZER, lcsc:BUZ-SMD_L9.6-W9.6-LS10.0-R, symbol ELRSFC:HND-9650B
- added C36, C37, C41, C44, C45, C46: 0.1uF, symbol Device:C
- added C38: 10nF, symbol Device:C
- added C39: 2.2uF, symbol Device:C
- added C40: 1uF, symbol Device:C
- added C42, C43: 12pF, symbol Device:C
- added D4: GREEN, symbol Device:LED
- added H1: ~, symbol ELRSFC:GPS
- added H2: ~, symbol ELRSFC:BATTERY
- added H3: ~, symbol ELRSFC:CAP
- added H4: ~, symbol ELRSFC:CAMERA
- added H5: ~, symbol ELRSFC:POWER
- added H6: ~, symbol ELRSFC:VTX
- added R10: 5.1k, symbol Device:R
- added R11: 47k, symbol Device:R
- added R12: 10k, symbol Device:R
- added R13: 120, symbol Device:R
- added U1: W25Q128JVSIQTR, lcsc:SOIC-8_L5.3-W5.3-P1.27-LS8.0-BL, symbol ELRSFC:W25Q128JVSIQTR
- added U5: MPU6500, lcsc:QFN-24_L3.0-W3.0-P0.40-BL-EP, symbol ELRSFC:MPU6500
- added U6: STM32F411CEU6, lcsc:UFQFPN-48_L7.0-W7.0-P0.50-BL-EP, symbol ELRSFC:STM32F411CEU6
- added X3: 25MHz, lcsc:CRYSTAL-SMD_4P-L3.2-W2.5-BL, symbol ELRSFC:X322525MOB4SI
- C1: value 2.2uF -> 10uF
- C14: value 1uF -> 10uF
- C15, C16, C18: value 0.1uF -> 10uF
- C17: value 0.1uF -> BULK
- C2: value 12pF -> 0.1uF
- C22: value 22uF -> 10uF
- C3: value 12pF -> 10uF
- R3: value 5.1k -> 10k
Connections:
- net +3v3: now also C1.1, C2.1, C37.2, C38.2, C40.1, C41.1, C44.1, C45.1, C46.1, H1.2 (3.3v), H5.2 (3.3v), R10.1, U1.3 (IO2), U1.7 (IO3), U1.8 (VCC), U5.13 (VDD), U5.8 (VDDIO), U6.24 (VDD), U6.36 (VDD), U6.48 (VDD), U6.49 (PAD), U6.9 (VDDA/VREF+); no longer C14.1, C15.1, C16.1, C17.1, C18.1, C19.1
- net +5V: now also C18.1, C19.1, H1.1 (5v), H4.1 (5v), H5.1 (5v)
- net BATTERY: now also C14.1, C15.1, C16.1, C17.1, C3.1, H2.1 (BATTERY), H3.1 (BATTERY), H6.1 (BATTERY), R11.1
- net GND: now also C20.2, R4.2, BUZZER1.2, C36.1, C37.1, C38.1, C39.2, C40.2, C41.2, C42.2, C43.2, C44.2, C45.2, C46.2, H1.3 (GND), H2.2 (GND), H3.2 (GND), H4.2 (GND), H5.3 (GND), H6.2 (GND), R12.2, U1.4 (GND), U5.11 (FSYNC), U5.18 (GND), U5.20 (RESV), U5.25 (EP), U6.23 (VSS), U6.35 (VSS), U6.47 (VSS), U6.8 (VSSA/VREF-), X3.2 (GND), X3.4 (GND); no longer C20.1, R4.1
- net NRST: now also U6.7 (NRST)
- net PB12: now also U6.25 (PB12)
- net PB13: now also U1.6 (CLK), U6.26 (PB13)
- net PB14: now also U1.2 (DO), U6.27 (PB14)
- net PB15: now also U1.5 (DI), U6.28 (PB15)
- net VIDIN: now also H4.3 (VID_IN)
- net VIDOUT: now also H6.3 (VID_OUT)
- net PB1: now reaches R3.2
- net PB1: now also U1.1 (~{CS}), U6.19 (PB1)
- new net: BUZZER1.1, R13.2
- new net: C43.1, U6.5 (PH0-OSC_IN), X3.1 (OSC1)
- new net: D4.2 (A), R10.2
- new net: C36.2, U5.10 (REGOUT)
- new net: D4.1 (K), U6.2 (PC13)
- new net: C39.1, U6.22 (VCAP1)
- new net: C42.1, U6.6 (PH1-OSC_OUT), X3.3 (OSC2)
- new net BOOT0: C20.1, R4.1, SW1.2, U6.44 (BOOT0)
- new net BYPASS: H4.4 (BYPASS), H6.4 (BYPASS)
- new net PA10: H1.5 (RX), U6.31 (PA10)
- new net PA4: U5.22 (nCS), U6.14 (PA4)
- new net PA5: U5.23 (SCL/SCLK), U6.15 (PA5)
- new net PA6: U5.9 (SDO/AD0), U6.16 (PA6)
- new net PA7: U5.24 (SDA/SDI), U6.17 (PA7)
- new net PA9: H1.4 (TX), U6.30 (PA9)
- new net PB0: R11.2, R12.1, U6.18 (PB0)
- new net PB2: R13.1, U6.20 (PB2)
- no-connect marks 17 -> 31
Other:
- note added: "FLASH"
- note added: "IMU"
- note added: "STM32"
- moved on the sheet: C20, C27, C28, C29, C30, C31, C32, C33, C34, C5, C6, C7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

Commit message: Sixth entry
Parts:
- removed C17: BULK, symbol Device:C
- removed C31, C33: 10uF, lcsc:CAP-SMD_L3.2-W1.6-RD-C7171, symbol ELRSFC:TAJA106K016RNJ
- removed D1: SS34, Diode_SMD:D_SMA, symbol Diode:SS34
- added D1: B5819W, ELRSFC:SOD-123_L2.7-W1.6-LS3.7-RD-1, symbol ELRSFC:B5819W_C8598
- added D2: USBLC6-2SC6, ELRSFC:SOT-23-6_L2.9-W1.6-P0.95-LS2.8-BL, symbol ELRSFC:USBLC6-2SC6
- added H7: SWD, ELRSFC:SWD, symbol ELRSFC:SWD
- added H8: ESC, ELRSFC:ESC, symbol ELRSFC:ESC
- added H9: RX, ELRSFC:RX, symbol ELRSFC:RX
- BUZZER1: footprint lcsc:BUZ-SMD_L9.6-W9.6-LS10.0-R -> ELRSFC:BUZ-SMD_L9.6-W9.6-LS10.0-R
- C1, C10, C11, C12, C13, C18, C19, C2, C20, C27, C28, C29, C34, C36, C37, C38, C39, C4, C40, C41, C42, C43, C44, C45, C46, C5, C6, C7, C8, C9: footprint (none) -> Capacitor_SMD:C_0402_1005Metric
- C14, C15, C16, C22, C3: footprint (none) -> Capacitor_SMD:C_0603_1608Metric
- C21, C35: footprint lcsc:CASE-B_3528 -> ELRSFC:CASE-B_3528
- C30, C32: value 10uF -> 22uF; footprint lcsc:CAP-SMD_L3.2-W1.6-RD-C7171 -> ELRSFC:CAP-SMD_L3.2-W1.6-RD-C7171
- D3, D4: footprint (none) -> LED_SMD:LED_0805_2012Metric
- H1: value ~ -> GPS; footprint (none) -> ELRSFC:GPS
- H2: value ~ -> BAT; footprint (none) -> ELRSFC:BAT
- H3: value ~ -> CAP; footprint (none) -> ELRSFC:CAP
- H4: value ~ -> CAM; footprint (none) -> ELRSFC:CAM
- H5: value ~ -> PWR; footprint (none) -> ELRSFC:PWR
- H6: value ~ -> VTX; footprint (none) -> ELRSFC:VTX
- L1: footprint (none) -> Inductor_SMD:L_Sunlord_SWPA8040S
- R1, R10, R11, R12, R13, R2, R3, R4, R5, R6, R7: footprint (none) -> Resistor_SMD:R_0402_1005Metric
- R8, R9: footprint (none) -> Resistor_SMD:R_0603_1608Metric
- SW1, SW2: footprint lcsc:SW-SMD_L3.9-W3.0-P4.45 -> ELRSFC:SW-SMD_L3.9-W3.0-P4.45
- U1: footprint lcsc:SOIC-8_L5.3-W5.3-P1.27-LS8.0-BL -> ELRSFC:SOIC-8_L5.3-W5.3-P1.27-LS8.0-BL
- U2: footprint lcsc:SOIC-8_L5.0-W4.0-P1.27-LS6.0-BL -> ELRSFC:SOIC-8_L5.0-W4.0-P1.27-LS6.0-BL
- U3: footprint lcsc:SOT-223-3_L6.5-W3.4-P2.30-LS7.0-BR -> ELRSFC:SOT-223-3_L6.5-W3.4-P2.30-LS7.0-BR
- U4: footprint lcsc:TSSOP-28_L9.7-W4.4-P0.65-LS6.4-BL-EP-2 -> ELRSFC:TSSOP-28_L9.7-W4.4-P0.65-LS6.4-BL-EP-2
- U5: footprint lcsc:QFN-24_L3.0-W3.0-P0.40-BL-EP -> ELRSFC:QFN-24_L3.0-W3.0-P0.40-BL-EP
- U6: footprint lcsc:UFQFPN-48_L7.0-W7.0-P0.50-BL-EP -> ELRSFC:UFQFPN-48_L7.0-W7.0-P0.50-BL-EP
- X2, X3: footprint lcsc:CRYSTAL-SMD_4P-L3.2-W2.5-BL -> ELRSFC:CRYSTAL-SMD_4P-L3.2-W2.5-BL
Connections:
- net +3v3: now also H1.4 (3.3v); no longer H1.2 (3.3v)
- net +5V: now also H1.3 (5v), D2.5, H9.1 (5v); no longer H1.1 (5v)
- net D+: now also U6.33 (PA12), D2.6; no longer USB1.6 (DP1), USB1.8 (DP2)
- net D-: now also U6.32 (PA11), D2.4; no longer USB1.5 (DN2), USB1.7 (DN1)
- net GND: now also H1.5 (GND), D1.2 (+), D2.2, H9.2 (GND); no longer H1.3 (GND)
- net NRST: now also H7.1 (NRST)
- net PA10: now also H1.7 (RX); no longer H1.5 (RX)
- net PA9: now also H1.6 (TX); no longer H1.4 (TX)
- net at L1.1, U2.2 (OUTPUT): now also D1.1 (-)
- net PA2: now reaches U6.12 (PA2)
- net PA2: now also H9.3 (TX)
- net PA3: now reaches U6.13 (PA3)
- net PA3: now also H9.4 (RX)
- net PA13: now reaches U6.34 (PA13)
- net PA13: now also H7.2 (SWDIO)
- net PA14: now reaches U6.37 (PA14)
- net PA14: now also H7.3 (SWCLK)
- net PB4: now reaches U6.40 (PB4)
- net PB4: now also H8.1 (MOT1)
- net PB5: now reaches U6.41 (PB5)
- net PB5: now also H8.2 (MOT2)
- net PB6: now reaches U6.42 (PB6)
- net PB6: now also H8.3 (MOT3)
- net PB7: now reaches U6.43 (PB7)
- net PB7: now also H8.4 (MOT4)
- net PB8: now reaches U6.45 (PB8)
- net PB8: now also H1.2 (SCL)
- net PB9: now reaches U6.46 (PB9)
- net PB9: now also H1.1 (SDA)
- new net DIN+: D2.1, USB1.6 (DP1), USB1.8 (DP2)
- new net DIN-: D2.3, USB1.5 (DN2), USB1.7 (DN1)
- no-connect marks 31 -> 37
Other:
- moved on the sheet: C18, C19, C32, H2, H3, H4, H5, H6, R8

Commit message: Seventh entry
Parts:
- added C17, C23, C47, C48, C50: 0.1uF, Capacitor_SMD:C_0402_1005Metric, symbol Device:C
- added C24, C26: 10nF, Capacitor_SMD:C_0402_1005Metric, symbol Device:C
- added C25: 470nF, Capacitor_SMD:C_0603_1608Metric, symbol Device:C
- added C31, C33: 10pF, Capacitor_SMD:C_0402_1005Metric, symbol Device:C
- added C49: 10uF, Capacitor_SMD:C_0402_1005Metric, symbol Device:C
- added FL1: 2450FM07D0034T, ELRSFC:FIL_2450FM07D0034T, symbol ELRSFC:2450FM07D0034T
- added J1: Conn_Coaxial_Small, Connector_Coaxial:U.FL_Hirose_U.FL-R-SMT-1_Vertical, symbol Connector:Conn_Coaxial_Small
- added JP1: ENA, ELRSFC:ENA, symbol Jumper:Jumper_2_Small_Open
- added JP2: FLASH, ELRSFC:FLASH, symbol Jumper:Jumper_2_Small_Open
- added R14: 12k, Resistor_SMD:R_0402_1005Metric, symbol Device:R
- added R15, R16: 10k, Resistor_SMD:R_0402_1005Metric, symbol Device:R
- added U7: ESP8285H16, ELRSFC:QFN-32_L5.0-W5.0-P0.50-TL-EP3.7, symbol ELRSFC:ESP8285H16
- added U8: SX1281IMLTRT, ELRSFC:QFN-24_L4.0-W4.0-P0.50-TL-EP2.6, symbol ELRSFC:SX1281IMLTRT
- added X1: 52MHz, ELRSFC:CRYSTAL-SMD_4P-L2.0-W1.6-BL, symbol ELRSFC:XC21M4-52.000-F10NNHPL
- added X4: 26MHz, ELRSFC:CRYSTAL-SMD_4P-L2.0-W1.6-BL, symbol ELRSFC:XL7EL89CMI-111YLC-26M
- SW1, SW2: footprint ELRSFC:SW-SMD_L3.9-W3.0-P4.45 -> ELRSFC:SW_TS-1187A-B-A-B
Connections:
- net +3v3: now also C17.1, C23.1, C47.2, C48.1, C49.1, R15.1, U7.1 (VDDA), U7.11 (VDDPST), U7.17 (VDDPST), U7.29 (VDDD), U7.3 (VDD3P3), U7.30 (VDDA), U7.4 (VDD3P3), U8.11 (VBAT_IO), U8.15 (VBAT); no longer U6.49 (PAD)
- net +5V: now also C27.1, C28.1, C29.1; no longer C27.2, C28.2, C29.2
- net GND: now also C27.2, C28.2, C29.2, U4.29 (EP), U6.49 (PAD), C17.2, C23.2, C24.2, C25.2, C26.2, C31.2, C33.2, C47.1, C48.2, C49.2, C50.2, FL1.2, FL1.4, J1.2 (Ext), JP1.1 (A), JP2.1 (A), R14.2, R16.2, U7.33 (GND), U8.13 (GND), U8.20 (GND), U8.21 (GND), U8.23 (GND), U8.24 (GND), U8.25 (EP), U8.5 (GND), X1.2 (GND), X1.4 (GND), X4.2 (GND), X4.4 (GND); no longer C27.1, C28.1, C29.1
- net PA2: now also U7.25 (U0RXD)
- net PA3: now also U7.26 (U0TXD)
- new net: FL1.3, J1.1 (In)
- new net: C31.1, U7.28 (XTAL_IN), X4.1
- new net: C50.1, JP1.2 (B), R15.2, U7.7 (CHIP_EN)
- new net: JP2.2 (B), U7.15 (GPIO0)
- new net: C33.1, U7.27 (XTAL_OUT), X4.3
- new net: R14.1, U7.31 (RES12K)
- new net: C26.1, U8.1 (VR_PA)
- new net: U8.4 (XTA), X1.1
- new net: U8.6 (XTB), X1.3
- new net DCC_FB: C24.1, C25.1, U8.12 (DCC_FB), U8.2 (VDD_IN)
- new net GPIO12: U7.10 (MTDI), U8.16 (MISO_TX)
- new net GPIO13: U7.12 (MTCK), U8.17 (MOSI_RX)
- new net GPIO14: U7.9 (MTMS), U8.18 (SCK_RTSN)
- new net GPIO15: R16.1, U7.13 (MTDO), U8.19 (NSS_CTS)
- new net GPIO2: U7.14 (GPIO2), U8.3 (NRESET)
- new net GPIO4: U7.16 (GPIO4), U8.8 (DIO1)
- new net GPIO5: U7.24 (GPIO5), U8.7 (BUSY)
- new net RFOUT: FL1.1, U8.22 (RFIO)
- no-connect marks 37 -> 51
Other:
- note added: "ELRS ESP8285"
- note added: "ELRS SX1281"
- moved on the sheet: C18, C19, H1, H2, H3, H4, H5, H6, H7, H8, H9

Commit message: Eight entry
Parts:
- J1: footprint Connector_Coaxial:U.FL_Hirose_U.FL-R-SMT-1_Vertical -> ELRSFC:UFL
Changed lines of the file:
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@@
 			)
 		)
-		(property "Footprint" "Connector_Coaxial:U.FL_Hirose_U.FL-R-SMT-1_Vertical"
+		(property "Footprint" "ELRSFC:UFL"
 			(at 149.86 243.84 0)
 			(effects

Commit message: Ninth entry
Parts:
- removed C18: 10uF, Capacitor_SMD:C_0402_1005Metric, symbol Device:C
- removed C19: 0.1uF, Capacitor_SMD:C_0402_1005Metric, symbol Device:C
- removed X2: 27MHz, ELRSFC:CRYSTAL-SMD_4P-L3.2-W2.5-BL, symbol ELRSFC:S3227000181040
- added X2: 27MHz, ELRSFC:CRYSTAL-SMD_4P-L2.0-W1.6-BL, symbol ELRSFC:7D027000Q01
Connections:
- net GND: now also X2.2 (GND), X2.4 (GND)
- net at U4.5 (CLKIN): now also X2.3
- net at U4.6 (XFB): now also X2.1
Changed lines of the file:
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@@
 	)
 	(junction
-		(at 93.98 212.09)
-		(diameter 0)
-		(color 0 0 0 0)
-	)
-	(junction
 		(at 24.13 110.49)
 		(diameter 0)
@@
 	)
 	(junction
-		(at 93.98 204.47)
-		(diameter 0)
-		(color 0 0 0 0)
-	)
-	(junction
 		(at 54.61 46.99)
 		(diameter 0)
@@
 	)
 	(junction
-		(at 87.63 204.47)
-		(diameter 0)
-		(color 0 0 0 0)
-	)
-	(junction
 		(at 270.51 147.32)
 		(diameter 0)
@@
 	)
 	(junction
-		(at 97.79 212.09)
-		(diameter 0)
-		(color 0 0 0 0)
-	)
-	(junction
 		(at 50.8 266.7)
 		(diameter 0)
@@
 	(wire
 		(pts
-			(xy 87.63 212.09) (xy 93.98 212.09)
-		)
-		(stroke
-			(width 0)
-			(type default)
-		)
-	)
-	(wire
-		(pts
 			(xy 17.78 36.83) (xy 17.78 41.91)
 		)
@@
 	(wire
 		(pts
-			(xy 87.63 204.47) (xy 93.98 204.47)
-		)
-		(stroke
-			(width 0)
-			(type default)
-		)
-	)
-	(wire
-		(pts
 			(xy 158.75 119.38) (xy 166.37 119.38)
 		)
@@
 	(wire
 		(pts
-			(xy 93.98 212.09) (xy 97.79 212.09)
-		)
-		(stroke
-			(width 0)
-			(type default)
-		)
-	)
-	(wire
-		(pts
 			(xy 317.5 222.25) (xy 335.28 222.25)
 		)
@@
 	(symbol
 		(lib_id "power:+5V")
-		(at 87.63 204.47 0)
+		(at 93.98 204.47 180)
 		(unit 1)
 		(exclude_from_sim no)
@@
 		(dnp no)
 		(property "Reference" "#PWR031"
-			(at 87.63 208.28 0)
+			(at 93.98 200.66 0)
 			(effects
 				(font
@@
 		)
 		(property "Value" "+5V"
-			(at 87.376 200.914 0)
+			(at 94.234 208.026 0)
 			(effects
 				(font
@@
 		)
 		(property "Footprint" ""
-			(at 87.63 204.47 0)
+			(at 93.98 204.47 0)
 			(effects
 				(font
@@
 		)
 		(property "Datasheet" ""
-			(at 87.63 204.47 0)
+			(at 93.98 204.47 0)
 			(effects
 				(font
@@
 		)
 		(property "Description" "Power symbol creates a global label with name \"+5V\""
-			(at 87.63 204.47 0)
+			(at 93.98 204.47 0)
 			(effects
 				(font
@@
 	)
 	(symbol
-		(lib_id "ELRSFC:S3227000181040")
-		(at 107.95 132.08 0)
-		(unit 1)
-		(exclude_from_sim no)
-		(in_bom yes)
-		(on_board yes)
-		(dnp no)
-		(property "Reference" "X2"
-			(at 107.696 125.984 0)
-			(effects
-				(font
-					(size 1.27 1.27)
-				)
-			)
-		)
-		(property "Value" "27MHz"
-			(at 107.696 138.176 0)
-			(effects
-				(font
-					(size 1.27 1.27)
-				)
-			)
-		)
-		(property "Footprint" "ELRSFC:CRYSTAL-SMD_4P-L3.2-W2.5-BL"
-			(at 107.95 142.24 0)
-			(effects
-				(font
-					(size 1.27 1.27)
-				)
-				(hide yes)
-			)
-		)
-		(property "Datasheet" "https://lcsc.com/product-detail/New-Arrivals_JGHC-S3227000181040_C390777.html"
-			(at 107.95 144.78 0)
-			(effects
-				(font
-					(size 1.27 1.27)
-				)
-				(hide yes)
-			)
-		)
-		(property "Description" ""
-			(at 107.95 132.08 0)
-			(effects
-				(font
-					(size 1.27 1.27)
-				)
-				(hide yes)
-			)
-		)
-		(property "LCSC Part" "C390777"
-			(at 107.95 147.32 0)
-			(effects
-				(font
-					(size 1.27 1.27)
-				)
-				(hide yes)
-			)
-		)
-		(pin "3"
-		)
-		(pin "1"
-		)
-		(pin "4"
-		)
-		(pin "2"
-		)
-		(instances
-			(project ""
-				(path "/42d441ea-c807-4e8f-bb94-f3987632e9a7"
-					(reference "X2")
-					(unit 1)
-				)
-			)
-		)
-	)
-	(symbol
 		(lib_id "Device:LED")
 		(at 151.13 57.15 180)
@@
 	)
 	(symbol
+		(lib_id "ELRSFC:7D027000Q01")
+		(at 107.95 132.08 0)
+		(unit 1)
+		(exclude_from_sim no)
+		(in_bom yes)
+		(on_board yes)
+		(dnp no)
+		(property "Reference" "X2"
+			(at 107.95 125.476 0)
+			(effects
+				(font
+					(size 1.27 1.27)
+				)
+			)
+		)
+		(property "Value" "27MHz"
+			(at 107.95 138.938 0)
+			(effects
+				(font
+					(size 1.27 1.27)
+				)
+			)
+		)
+		(property "Footprint" "ELRSFC:CRYSTAL-SMD_4P-L2.0-W1.6-BL"
+			(at 107.95 142.24 0)
+			(effects
+				(font
+					(size 1.27 1.27)
+				)
+				(hide yes)
+			)
+		)
+		(property "Datasheet" "https://lcsc.com/product-detail/SMD-Crystal-Resonators_HD-7D027000Q01_C648952.html"
+			(at 107.95 144.78 0)
+			(effects
+				(font
+					(size 1.27 1.27)
+				)
+				(hide yes)
+			)
+		)
+		(property "Description" ""
+			(at 107.95 132.08 0)
+			(effects
+				(font
+					(size 1.27 1.27)
+				)
+				(hide yes)
+			)
+		)
+		(property "LCSC Part" "C648952"
+			(at 107.95 147.32 0)
+			(effects
+				(font
+					(size 1.27 1.27)
+				)
+				(hide yes)
+			)
+		)
+		(pin "1"
+		)
+		(pin "2"
+		)
+		(pin "4"
+		)
+		(pin "3"
+		)
+		(instances
+			(project ""
+				(path "/42d441ea-c807-4e8f-bb94-f3987632e9a7"
+					(reference "X2")
+					(unit 1)
+				)
+			)
+		)
+	)
+	(symbol
 		(lib_id "power:+5V")
 		(at 45.72 52.07 270)
@@
 	)
 	(symbol
-		(lib_id "Device:C")
-		(at 93.98 208.28 0)
-		(mirror y)
-		(unit 1)
-		(exclude_from_sim no)
-		(in_bom yes)
-		(on_board yes)
-		(dnp no)
-		(property "Reference" "C19"
-			(at 93.726 206.248 0)
-			(effects
-				(font
-					(size 1.27 1.27)
-				)
-				(justify left)
-			)
-		)
-		(property "Value" "0.1uF"
-			(at 93.472 211.328 0)
-			(effects
-				(font
-					(size 1.27 1.27)
-				)
-				(justify left)
-			)
-		)
-		(property "Footprint" "Capacitor_SMD:C_0402_1005Metric"
-			(at 93.0148 212.09 0)
-			(effects
-				(font
-					(size 1.27 1.27)
-				)
-				(hide yes)
-			)
-		)
-		(property "Datasheet" "~"
-			(at 93.98 208.28 0)
-			(effects
-				(font
-					(size 1.27 1.27)
-				)
-				(hide yes)
-			)
-		)
-		(property "Description" "Unpolarized capacitor"
-			(at 93.98 208.28 0)
-			(effects
-				(font
-					(size 1.27 1.27)
-				)
-				(hide yes)
-			)
-		)
-		(pin "2"
-		)
-		(pin "1"
-		)
-		(instances
-			(project "ELRSFC"
-				(path "/42d441ea-c807-4e8f-bb94-f3987632e9a7"
-					(reference "C19")
-					(unit 1)
-				)
-			)
-		)
-	)
-	(symbol
 		(lib_id "Device:R")
 		(at 321.31 214.63 90)
@@
 					(unit 1)
 				)
-			)
-		)
-	)
-	(symbol
-		(lib_id "Device:C")
-		(at 87.63 208.28 0)
-		(mirror y)
-		(unit 1)
-		(exclude_from_sim no)
-		(in_bom yes)
-		(on_board yes)
-		(dnp no)
-		(property "Reference" "C18"
-			(at 87.376 206.248 0)
-			(effects
-				(font
-					(size 1.27 1.27)
-				)
-				(justify left)
-			)
-		)
-		(property "Value" "10uF"
-			(at 87.122 211.328 0)
-			(effects
-				(font
-					(size 1.27 1.27)
-				)
-				(justify left)
-			)
-		)
-		(property "Footprint" "Capacitor_SMD:C_0402_1005Metric"
-			(at 86.6648 212.09 0)
-			(effects
-				(font
-					(size 1.27 1.27)
-				)
-				(hide yes)
-			)
-		)
-		(property "Datasheet" "~"
-			(at 87.63 208.28 0)
-			(effects
-				(font
-					(size 1.27 1.27)
-				)
-				(hide yes)
-			)
-		)
-		(property "Description" "Unpolarized capacitor"
-			(at 87.63 208.28 0)
-			(effects
-				(font
-					(size 1.27 1.27)
-				)
-				(hide yes)
-			)
-		)
-		(pin "2"
-		)
-		(pin "1"
-		)
-		(instances
-			(project "ELRSFC"
-				(path "/42d441ea-c807-4e8f-bb94-f3987632e9a7"
-					(reference "C18")
-					(unit 1)
-				)

Commit message: high cortisol
Parts:
- removed C14, C15, C16, C22, C3: 10uF, Capacitor_SMD:C_0603_1608Metric, symbol Device:C
- removed C20, C46, C6, C9: 0.1uF, Capacitor_SMD:C_0402_1005Metric, symbol Device:C
- removed H9: RX, ELRSFC:RX, symbol ELRSFC:RX
- removed SW1, SW2: SWITCH, ELRSFC:SW_TS-1187A-B-A-B, symbol ELRSFC:TS-1088-AR02016
- removed U3: AMS1117-3.3, ELRSFC:SOT-223-3_L6.5-W3.4-P2.30-LS7.0-BR, symbol ELRSFC:AMS1117-3.3
- added C18: 10nF, Capacitor_SMD:C_0402_1005Metric, symbol Device:C
- added U9: SPX3819M5-L-3-3/TR, ELRSFC:SOT-23-5_L3.0-W1.7-P0.95-LS2.8-BL, symbol ELRSFC:SPX3819M5-L-3-3_TR
- C5: footprint Capacitor_SMD:C_0402_1005Metric -> Capacitor_SMD:C_0603_1608Metric
- R4, R7: footprint Resistor_SMD:R_0402_1005Metric -> Resistor_SMD:R_0603_1608Metric
Connections:
- net +3v3: now also U9.5 (OUT)
- net +5V: now also U9.1 (IN), U9.3 (EN)
- net BOOT0: now also H7.1 (BOOT)
- net GND: now also C18.2, U9.2 (GND)
- net NRST: now also H7.2 (NRST); no longer H7.1 (NRST)
- net PA13: now also H7.3 (SWDIO); no longer H7.2 (SWDIO)
- net PA14: now also H7.4 (SWCLK); no longer H7.3 (SWCLK)
- net at U6.2 (PC13): no longer D4.1 (K)
- net at U6.29 (PA8): now also D4.1 (K)
- new net: C18.1, U9.4 (BYP)
Other:
- moved on the sheet: BUZZER1, C5, C7, C8, D4, R10, R13, R4

Commit message: (hopefully) finalized PCB
Parts:
- added D5: 1N4148W, Diode_SMD:D_SOD-123, symbol Diode:1N4148W
- added H10: SENSE, ELRSFC:SENSE, symbol ELRSFC:SENSE
- added H9: EXTRA, ELRSFC:EXTRA, symbol ELRSFC:EXTRA
- added Q1: 2N7002, Package_TO_SOT_SMD:SOT-23, symbol Transistor_FET:2N7002
- added R17: 10k, Resistor_SMD:R_0402_1005Metric, symbol Device:R
- C1, C10, C13, C49, C7, C8: LCSC Part (none) -> C15525
- C11, C17, C2, C23, C27, C28, C29, C34, C36, C37, C4, C41, C44, C45, C47, C48, C50: LCSC Part (none) -> C307331
- C12, C18, C24, C26, C38: LCSC Part (none) -> C15195
- C25: LCSC Part (none) -> C1623
- C30, C32: LCSC Part C7171 -> (none)
- C31, C33: LCSC Part (none) -> C32949
- C39: LCSC Part (none) -> C12530
- C40: LCSC Part (none) -> C52923
- C42, C43: LCSC Part (none) -> C1547
- D3: LCSC Part (none) -> C84256
- D4: LCSC Part (none) -> C2297
- R1, R10, R2, R6: LCSC Part (none) -> C25905
- R11: LCSC Part (none) -> C25792
- R12, R15, R16, R3, R5: LCSC Part (none) -> C25744
- R13: LCSC Part (none) -> C25079
- R14: LCSC Part (none) -> C25752
- R8, R9: LCSC Part (none) -> C4275
Connections:
- net +3v3: now also BUZZER1.1, D5.1 (K)
- net GND: now also Q1.2 (S), R17.2; no longer BUZZER1.2
- net PB1: now also H10.1 (SENSE); no longer R3.2, U1.1 (~{CS})
- net PB2: now also R17.1
- net at R13.2: now also Q1.1 (G); no longer BUZZER1.1
- net PB10: now reaches U6.21 (PB10)
- net PB10: now also R3.2, U1.1 (~{CS})
- net PA15: now reaches U6.38 (PA15)
- net PA15: now also H9.1 (XTRA)
- new net: BUZZER1.2, D5.2 (A), Q1.3 (D)
- no-connect marks 51 -> 49
Other:
- moved on the sheet: BUZZER1, R13
